Commit message: it's working ig

File: body.urdf (robot description, URDF)
Before this commit: robot robot, 9 links, 8 joints
Links:
- removed link BackLeg
- removed link BackLower
- removed link FrontLeg
- removed link FrontLower
- removed link LeftLeg
- removed link LeftLower
- removed link RightLeg
- removed link RightLower
- added link lower-back-left, mass 1; collision box size=0.2 0.2 1; visual box size=0.2 0.2 1
- added link lower-back-right, mass 1; collision box size=0.2 0.2 1; visual box size=0.2 0.2 1
- added link lower-front-left, mass 1; collision box size=0.2 0.2 1; visual box size=0.2 0.2 1
- added link lower-front-right, mass 1; collision box size=0.2 0.2 1; visual box size=0.2 0.2 1
- added link upper-back-left, mass 1; collision box size=0.2 1 0.2; visual box size=0.2 1 0.2
- added link upper-back-right, mass 1; collision box size=1 0.2 0.2; visual box size=1 0.2 0.2
- added link upper-front-left, mass 1; collision box size=0.2 1 0.2; visual box size=0.2 1 0.2
- added link upper-front-right, mass 1; collision box size=1 0.2 0.2; visual box size=1 0.2 0.2
Joints:
- removed joint BackLeg_BackLower
- removed joint FrontLeg_FrontLower
- removed joint LeftLeg_LeftLower
- removed joint RightLeg_RightLower
- removed joint Torso_BackLeg
- removed joint Torso_FrontLeg
- removed joint Torso_LeftLeg
- removed joint Torso_RightLeg
- added joint Torso_upper-back-left: type revolute, parent Torso, child upper-back-left, origin xyz=0 -0.5 1 rpy=0 0 0, axis 1 0 0, limit lower=-3.14159 upper=3.14159 effort=0.0 velocity=0.0
- added joint Torso_upper-back-right: type revolute, parent Torso, child upper-back-right, origin xyz=0.5 0 1 rpy=0 0 0, axis 0 1 0, limit lower=-3.14159 upper=3.14159 effort=0.0 velocity=0.0
- added joint Torso_upper-front-left: type revolute, parent Torso, child upper-front-left, origin xyz=0 0.5 1 rpy=0 0 0, axis 1 0 0, limit lower=-3.14159 upper=3.14159 effort=0.0 velocity=0.0
- added joint Torso_upper-front-right: type revolute, parent Torso, child upper-front-right, origin xyz=-0.5 0 1 rpy=0 0 0, axis 0 1 0, limit lower=-3.14159 upper=3.14159 effort=0.0 velocity=0.0
- added joint upper-back-left_lower-back-left: type revolute, parent upper-back-left, child lower-back-left, origin xyz=0 -1 0 rpy=0 0 0, axis 1 0 0, limit lower=-3.14159 upper=3.14159 effort=0.0 velocity=0.0
- added joint upper-back-right_lower-back-right: type revolute, parent upper-back-right, child lower-back-right, origin xyz=1 0 0 rpy=0 0 0, axis 0 1 0, limit lower=-3.14159 upper=3.14159 effort=0.0 velocity=0.0
- added joint upper-front-left_lower-front-left: type revolute, parent upper-front-left, child lower-front-left, origin xyz=0 1 0 rpy=0 0 0, axis 1 0 0, limit lower=-3.14159 upper=3.14159 effort=0.0 velocity=0.0
- added joint upper-front-right_lower-front-right: type revolute, parent upper-front-right, child lower-front-right, origin xyz=-1 0 0 rpy=0 0 0, axis 0 1 0, limit lower=-3.14159 upper=3.14159 effort=0.0 velocity=0.0
